File: de0-cv-shield.sch (KiCad schematic (older format))
At the start: 30 parts, among them P101 USB_OTG, P102 CONN_02X20, U101 ISL89410, U102 ISL89410, U103 FT230XS, U104 STM32F373CCTx, U105 MCP2562-E/SN, U106 LD1117S33TR, U107 MAX9924

Commit message: Fix wrong FTDI wiring, add silk board label
Connections:
- net ftdi_rx: now also U104.45 (CAN_RX/CEC/COMP1_OUT/I2C1_SCL/I2S2_CK/SPI2_SCK/TIM16_CH1/TIM19_CH3/TIM4_CH3/TSC_SYNC/USART3_TX/PB8); no longer U104.46 (CAN_TX/COMP2_OUT/DAC1_EXTI9/DAC2_EXTI9/I2C1_SDA/I2S2_WS/IR_OUT/SPI2_NSS/TIM17_CH1/TIM19_CH4/TIM4_CH4/USART3_RX/PB9)
- net ftdi_tx: now also U104.46 (CAN_TX/COMP2_OUT/DAC1_EXTI9/DAC2_EXTI9/I2C1_SDA/I2S2_WS/IR_OUT/SPI2_NSS/TIM17_CH1/TIM19_CH4/TIM4_CH4/USART3_RX/PB9); no longer U104.45 (CAN_RX/CEC/COMP1_OUT/I2C1_SCL/I2S2_CK/SPI2_SCK/TIM16_CH1/TIM19_CH3/TIM4_CH3/TSC_SYNC/USART3_TX/PB8)
- net at U103.14 (CBUS1): now also D101.1 (K); no longer D102.1 (K)
- net at U103.15 (CBUS0): no longer D101.1 (K)
- net at U103.7 (CBUS2): now also D102.1 (K)
Changed lines of the file:
@@
 Text GLabel 5850 9750 2    60   Input ~ 0
 ftdi_rx
+Text GLabel 13500 4200 2    60   Input ~ 0
+ftdi_rx
 Text GLabel 13500 4300 2    60   Input ~ 0
-ftdi_rx
-Text GLabel 13500 4200 2    60   Input ~ 0
 ftdi_tx
 $Comp
@@
 NoConn ~ 4200 9650
 NoConn ~ 3850 9850
-NoConn ~ 5600 10350
 NoConn ~ 5600 10450
 $Sheet
@@
 	172050 -111600 162200 -111600
 Wire Wire Line
-	6550 10050 6550 10150
-Wire Wire Line
-	6550 10150 5600 10150
-Wire Wire Line
-	5600 10250 6900 10250
-Wire Wire Line
-	6900 10250 6900 10050
+	6550 10050 6550 10250
+Wire Wire Line
+	6900 10050 6900 10350
 Wire Wire Line
 	6550 9150 6550 9250
@@
 Wire Wire Line
 	2700 10800 2700 10950
-Wire Wire Line
-	13500 4200 13300 4200
-Wire Wire Line
-	13500 4300 13300 4300
 Wire Wire Line
 	9950 10350 9950 10400
@@
 Wire Wire Line
 	18750 10800 18750 10850
+Wire Wire Line
+	6550 10250 5600 10250
+Wire Wire Line
+	6900 10350 5600 10350
+NoConn ~ 5600 10150
+Wire Wire Line
+	13500 4200 13300 4200
+Wire Wire Line
+	13300 4300 13500 4300
 $EndSCHEMATC
